File: kicad6_pcb/CSA+Amp.kicad_sch (KiCad schematic)
At the start: 24 parts, among them J301 CA probe, J302 RV Prob, U301 CR110, U302 TL071

Commit message: CSA carrier v2. Multiple fixes and improvements.
Parts:
- added C309: Open, Capacitor_SMD:C_0805_2012Metric_Pad1.18x1.45mm_HandSolder, symbol Device:C_Small
- C301: footprint Capacitor_SMD:C_2220_5650Metric_Pad1.97x5.40mm_HandSolder -> Capacitor_SMD:C_1206_3216Metric_Pad1.33x1.80mm_HandSolder; Mouser 810-CGA9N4C0G2W104JA -> 80-C1206C104K3HAUTO
- C302: footprint Capacitor_SMD:C_2220_5650Metric_Pad1.97x5.40mm_HandSolder -> Capacitor_THT:C_Disc_D5.0mm_W2.5mm_P5.00mm; Mouser 810-CGA9N4C0G2W104JA -> 810-FA26C0G2J103JNU6
- U301: Mouser 575-8019300810012000 -> 575-8019300810012000
- U302: footprint Package_SO:SOIC-8_5.23x5.23mm_P1.27mm -> Package_SO:SOIC-8_3.9x4.9mm_P1.27mm
- renumbered RV301 to Rv301
Connections:
- net Out: now also C309.1
- net at R307.1, R308.2, U302.2 (-): now also C309.2
Changed lines of the file:
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@@
   (junction (at 76.2 58.42) (diameter 0) (color 0 0 0 0)
   )
+  (junction (at 217.17 127) (diameter 0) (color 0 0 0 0)
+  )
   (junction (at 135.89 109.22) (diameter 0) (color 0 0 0 0)
   )
   (junction (at 166.37 124.46) (diameter 0) (color 0 0 0 0)
+  )
+  (junction (at 217.17 137.16) (diameter 0) (color 0 0 0 0)
   )
   (junction (at 83.82 82.55) (diameter 0) (color 0 0 0 0)
@@
     (stroke (width 0) (type default) (color 0 0 0 0))
   )
+  (wire (pts (xy 217.17 127) (xy 217.17 129.54))
+    (stroke (width 0) (type default) (color 0 0 0 0))
+  )
   (wire (pts (xy 232.41 156.21) (xy 232.41 151.13))
     (stroke (width 0) (type default) (color 0 0 0 0))
@@
     (stroke (width 0) (type default) (color 0 0 0 0))
   )
+  (wire (pts (xy 217.17 134.62) (xy 217.17 137.16))
+    (stroke (width 0) (type default) (color 0 0 0 0))
+  )
   (wire (pts (xy 220.98 146.05) (xy 232.41 146.05))
     (stroke (width 0) (type default) (color 0 0 0 0))
@@
     (stroke (width 0) (type default) (color 0 0 0 0))
   )
+  (wire (pts (xy 217.17 127) (xy 220.98 127))
+    (stroke (width 0) (type default) (color 0 0 0 0))
+  )
   (wire (pts (xy 135.89 109.22) (xy 135.89 114.3))
     (stroke (width 0) (type default) (color 0 0 0 0))
@@
     (stroke (width 0) (type default) (color 0 0 0 0))
   )
-  (wire (pts (xy 212.09 127) (xy 220.98 127))
+  (wire (pts (xy 212.09 127) (xy 217.17 127))
     (stroke (width 0) (type default) (color 0 0 0 0))
   )
@@
     (pin "2")
   )
+  (symbol (lib_id "Device:C_Small") (at 217.17 132.08 0) (unit 1)
+    (in_bom yes) (on_board yes)
+    (property "Reference" "C309" (id 0) (at 213.36 130.81 90))
+    (property "Value" "Open" (id 1) (at 210.82 130.81 90))
+    (property "Footprint" "Capacitor_SMD:C_0805_2012Metric_Pad1.18x1.45mm_HandSolder" (id 2) (at 217.17 132.08 0)
+      (effects (font (size 1.27 1.27)) hide)
+    )
+    (property "Datasheet" "" (id 3) (at 217.17 132.08 0)
+      (effects (font (size 1.27 1.27)) hide)
+    )
+    (property "Digikey" "" (id 4) (at 217.17 132.08 0)
+      (effects (font (size 1.27 1.27)) hide)
+    )
+    (property "Mouser" "80-C0805C104K5RACLR " (id 5) (at 217.17 132.08 0)
+      (effects (font (size 1.27 1.27)) hide)
+    )
+    (pin "1")
+    (pin "2")
+  )
   (symbol (lib_id "Device:C_Small") (at 113.03 87.63 180) (unit 1)
     (in_bom yes) (on_board yes)
@@
   (symbol (lib_id "Device:R_Potentiometer_Trim") (at 220.98 151.13 90) (unit 1)
     (in_bom yes) (on_board yes) (fields_autoplaced)
-    (property "Reference" "RV301" (id 0) (at 220.98 154.94 90))
+    (property "Reference" "Rv301" (id 0) (at 220.98 154.94 90))
     (property "Value" "10k" (id 1) (at 220.98 157.48 90))
     (property "Footprint" "Potentiometer_THT:Potentiometer_Bourns_3266W_Vertical" (id 2) (at 220.98 151.13 0)
@@
     (property "Reference" "U302" (id 0) (at 198.12 119.38 0))
     (property "Value" "TL071" (id 1) (at 210.82 123.19 0))
-    (property "Footprint" "Package_SO:SOIC-8_5.23x5.23mm_P1.27mm" (id 2) (at 205.74 125.73 0)
+    (property "Footprint" "Package_SO:SOIC-8_3.9x4.9mm_P1.27mm" (id 2) (at 205.74 125.73 0)
       (effects (font (size 1.27 1.27)) hide)
     )
@@
       (effects (font (size 1.27 1.27)) hide)
     )
-    (property "Datasheet" "" (id 3) (at 204.47 138.43 0)
+    (property "Datasheet" "https://www.mouser.com/ProductDetail/KEMET/C0805C104K5RAC7411?qs=jbRM9o5BbzPcVXF0wW9AYg%3D%3D" (id 3) (at 204.47 138.43 0)
       (effects (font (size 1.27 1.27)) hide)
     )
@@
       (effects (font (size 1.27 1.27)) hide)
     )
-    (property "Mouser" " 575-8019300810012000 " (id 4) (at 129.54 115.57 0)
+    (property "Mouser" "575-8019300810012000 " (id 4) (at 129.54 115.57 0)
       (effects (font (size 1.27 1.27)) hide)
     )
@@
       (effects (font (size 1.27 1.27)) (justify right))
     )
-    (property "Footprint" "Capacitor_SMD:C_2220_5650Metric_Pad1.97x5.40mm_HandSolder" (id 2) (at 75.2348 60.96 0)
-      (effects (font (size 1.27 1.27)) hide)
-    )
-    (property "Datasheet" "https://product.tdk.com/system/files/dam/doc/product/capacitor/ceramic/mlcc/catalog/mlcc_automotive_midvoltage_en.pdf?ref_disty=mouser" (id 3) (at 76.2 64.77 0)
-      (effects (font (size 1.27 1.27)) hide)
-    )
-    (property "Mouser" "810-CGA9N4C0G2W104JA" (id 4) (at 76.2 64.77 0)
+    (property "Footprint" "Capacitor_SMD:C_1206_3216Metric_Pad1.33x1.80mm_HandSolder" (id 2) (at 75.2348 60.96 0)
+      (effects (font (size 1.27 1.27)) hide)
+    )
+    (property "Datasheet" "https://www.mouser.com/datasheet/2/212/KEM_C1007_X8R_ULTRA_150C_SMD-1102703.pdf" (id 3) (at 76.2 64.77 0)
+      (effects (font (size 1.27 1.27)) hide)
+    )
+    (property "Mouser" "80-C1206C104K3HAUTO" (id 4) (at 76.2 64.77 0)
       (effects (font (size 1.27 1.27)) hide)
     )
@@
     (property "Reference" "C302" (id 0) (at 92.71 76.2 90))
     (property "Value" "10n" (id 1) (at 92.71 78.74 90))
-    (property "Footprint" "Capacitor_SMD:C_2220_5650Metric_Pad1.97x5.40mm_HandSolder" (id 2) (at 96.52 81.5848 0)
-      (effects (font (size 1.27 1.27)) hide)
-    )
-    (property "Datasheet" "https://product.tdk.com/system/files/dam/doc/product/capacitor/ceramic/mlcc/catalog/mlcc_automotive_midvoltage_en.pdf?ref_disty=mouser" (id 3) (at 92.71 82.55 0)
-      (effects (font (size 1.27 1.27)) hide)
-    )
-    (property "Mouser" "810-CGA9N4C0G2W104JA" (id 4) (at 92.71 82.55 0)
+    (property "Footprint" "Capacitor_THT:C_Disc_D5.0mm_W2.5mm_P5.00mm" (id 2) (at 96.52 81.5848 0)
+      (effects (font (size 1.27 1.27)) hide)
+    )
+    (property "Datasheet" "https://product.tdk.com/system/files/dam/doc/product/capacitor/ceramic/lead-mlcc/catalog/leadmlcc_halogenfree_fa_en.pdf?ref_disty=mouser" (id 3) (at 92.71 82.55 0)
+      (effects (font (size 1.27 1.27)) hide)
+    )
+    (property "Mouser" "810-FA26C0G2J103JNU6 " (id 4) (at 92.71 82.55 0)
       (effects (font (size 1.27 1.27)) hide)
     )
@@
       (effects (font (size 1.27 1.27)) hide)
     )
-    (property "Datasheet" "" (id 3) (at 204.47 114.3 0)
-      (effects (font (size 1.27 1.27)) hide)
-    )
+    (property "Datasheet" "https://www.mouser.com/ProductDetail/KEMET/C0805C104K5RAC7411?qs=jbRM9o5BbzPcVXF0wW9AYg%3D%3D" (id 3) (at 204.47 114.3 0)
+      (effects (font (size 1.27 1.27)) hide)
+    )
